Commit message: update urdf for two wheel robot

File: urdf/slam_bot.xacro (robot description, xacro)
@@ -1,5 +1,5 @@
 <?xml version='1.0'?>
-<robot name="slam_bot" xmlns:xacro="http://www.ros.org/wiki/xacro">
-<xacro:include filename="$(find slam_project)/urdf/slam_bot.gazebo" />
+<robot name="udacity_bot" xmlns:xacro="http://www.ros.org/wiki/xacro">
+<xacro:include filename="$(find udacity_bot)/urdf/udacity_bot.gazebo" />
   <link name="robot_footprint"></link>
   <joint name="robot_footprint_joint" type="fixed">
@@ -11,5 +11,5 @@
     <pose>0 0 0.1 0 0 0</pose>
     <inertial>
-      <mass value="25.0"/>
+      <mass value="15.0"/>
       <origin xyz="0.0 0 0" rpy=" 0 0 0"/>
       <inertia ixx="0.1" ixy="0" ixz="0" iyy="0.1" iyz="0" izz="0.1" />
@@ -27,5 +27,5 @@
       </geometry>
     </visual>
-   <!--  <collision name='back_caster_collision'>
+    <collision name='back_caster_collision'>
       <origin xyz="-0.15 0 -0.05" rpy=" 0 0 0"/>
       <geometry>
@@ -51,7 +51,62 @@
       </geometry>
     </visual>
- -->
   </link>
   <!-- Added wheels to the chessis -->
+  <link name='left_wheel'>
+    <inertial>
+      <mass value="5.0"/>
+      <origin xyz="0 0 0" rpy="0 1.5707 1.5707"/>
+      <inertia ixx="0.1" ixy="0" ixz="0" iyy="0.1" iyz="0" izz="0.1" />
+    </inertial>
+    <collision name='collision'>
+      <origin xyz="0 0 0" rpy="0 1.5707 1.5707"/>
+      <geometry>
+        <cylinder radius="0.1" length=".05"/>
+      </geometry>
+    </collision>
+    <visual name='left_wheel_visual'>
+      <origin xyz="0 0 0" rpy=" 0 1.5707 1.5707"/>
+      <geometry>
+        <cylinder radius="0.1" length=".05"/>
+      </geometry>
+    </visual>
+  </link>
+  <joint type="continuous" name="left_wheel_hinge">
+    <origin xyz="0.0 0.15 0.0" rpy="0 0 0"/>
+    <child link="left_wheel"/>
+    <parent link="chassis"/>
+    <axis xyz="0 1 0" rpy="0 0 0"/>
+    <limit effort="10000" velocity="1000"/>
+    <joint_properties damping="1.0" friction="1.0"/>
+  </joint>
+  <link name='right_wheel'>
+    <inertial>
+      <mass value="5.0"/>
+      <origin xyz="0 0 0" rpy="0 1.5707 1.5707"/>
+      <inertia ixx="0.1" ixy="0" ixz="0" iyy="0.1" iyz="0" izz="0.1" />
+    </inertial>
+    <collision name='collision'>
+      <origin xyz="0 0 0" rpy="0 1.5707 1.5707"/>
+      <geometry>
+        <cylinder radius="0.1" length=".05"/>
+      </geometry>
+    </collision>
+    <visual name='right_wheel_visual'>
+      <origin xyz="0 0 0" rpy=" 0 1.5707 1.5707"/>
+      <geometry>
+        <cylinder radius="0.1" length=".05"/>
+      </geometry>
+    </visual>
+  </link>
+  <joint type="continuous" name="right_wheel_hinge">
+    <origin xyz="0.0 -0.15 0.0" rpy="0 0 0"/>
+    <child link="right_wheel"/>
+    <parent link="chassis"/>
+    <axis xyz="0 1 0" rpy="0 0 0"/>
+    <limit effort="10000" velocity="1000"/>
+    <joint_properties damping="1.0" friction="1.0"/>
+  </joint>
+  <!-- Added four wheels to the chessis -->
+<!--
   <link name='front_left_wheel'>
     <inertial>
@@ -162,6 +217,42 @@
     <joint_properties damping="1.0" friction="1.0"/>
   </joint>
-  <!-- Added camera to the chessis -->
-  <link name='camera'>
+ -->
+ <!-- Added camera to the chessis -->
+  <link name="camera">
+      <origin>0 0 0 0 0 0</origin>
+      <inertial>
+        <origin xyz="0 0 0" rpy="3.14 0 0"/>
+        <mass value ="0.1"/>
+        <inertia ixx="1e-6" ixy="0" ixz="0" iyy="1e-6" iyz="0" izz="1e-6"/>
+      </inertial>
+      <collision name="collision">
+        <origin xyz="0 0 0" rpy="3.14 0 0"/>
+        <geometry>
+          <box size="0.05 0.05 0.05" />
+        </geometry>
+      </collision>
+      <visual>
+        <geometry>
+          <mesh filename="package://slam_project/meshes/kinect/meshes/kinect.dae" />
+        </geometry>
+      </visual>
+    </link>
+    <joint type="fixed" name="camera_joint">
+      <origin xyz="0.3 0 0" rpy="0 0 0" />
+      <child link="camera" />
+      <parent link="chassis" />
+    </joint>
+    <joint name="camera_optical_joint" type="fixed">
+      <!-- these values have to be these values otherwise the gazebo camera
+          image won't be aligned properly with the frame it is supposedly
+          originating from -->
+      <origin xyz="0 0 0" rpy="${-pi/2} 0 ${-pi/2}"/>
+      <parent link="camera"/>
+      <child link="camera_optical_link"/>
+    </joint>
+    <link name="camera_optical_link">
+  </link>
+  <!-- Added hokuyo(LIDAR) to the chessis -->
+  <link name='hokuyo'>
     <inertial>
       <mass value="0.1"/>
@@ -172,42 +263,17 @@
       <origin xyz="0 0 0" rpy="0 0 0"/>
       <geometry>
-        <box size="0.05 0.05 0.05"/>
-      </geometry>
-    </collision>
-    <visual name='camera_visual'>
-      <origin xyz="0 0 0" rpy="0 0 0"/>
-      <geometry>
-        <box size="0.05 0.05 0.05"/>
-      </geometry>
-    </visual>
-  </link>
-  <joint type="fixed" name="camera_joint">
-    <origin xyz="0.2 0 0" rpy="0 0 0"/>
-    <child link="camera"/>
-    <parent link="chassis"/>
-  </joint>
-<!-- Added hokuyo(LIDAR) to the chessis -->
-     <link name='hokuyo'>
-      <inertial>
-        <mass value="0.1"/>
-        <origin xyz="0 0 0" rpy="0 0 0"/>
-        <inertia ixx="1e-6" ixy="0" ixz="0" iyy="1e-6" iyz="0" izz="1e-6" />
-      </inertial>
-      <collision name='collision'>
-        <origin xyz="0 0 0" rpy="0 0 0"/>
-        <geometry>
-          <box size="0.01 0.01 0.01"/>
-        </geometry>
-      </collision>
-      <visual name='hokuyo_visual'>
-        <geometry>
-          <mesh filename="package://slam_project/meshes/hokuyo.dae" />
-        </geometry>
-      </visual>
-    </link>
-    <joint type="fixed" name="hokuyo_joint">
-      <origin xyz="0.15 0 0.1" rpy="0 0 0"/>
-      <child link="hokuyo"/>
-      <parent link="chassis"/>
-    </joint>
+        <box size="0.01 0.01 0.01"/>
+      </geometry>
+    </collision>
+    <visual name='hokuyo_visual'>
+      <geometry>
+        <mesh filename="package://udacity_bot/meshes/hokuyo.dae" />
+      </geometry>
+    </visual>
+  </link>
+  <joint type="fixed" name="hokuyo_joint">
+    <origin xyz="0.15 0 0.1" rpy="0 0 0"/>
+    <child link="hokuyo"/>
+    <parent link="chassis"/>
+  </joint>
 </robot>

Commit message: update urdf for slam_bot

File: urdf/slam_bot.xacro (robot description, xacro)
@@ -1,5 +1,5 @@
 <?xml version='1.0'?>
-<robot name="udacity_bot" xmlns:xacro="http://www.ros.org/wiki/xacro">
-<xacro:include filename="$(find udacity_bot)/urdf/udacity_bot.gazebo" />
+<robot name="slam_bot" xmlns:xacro="http://www.ros.org/wiki/xacro">
+<xacro:include filename="$(find slam_project)/urdf/slam_bot.gazebo" />
   <link name="robot_footprint"></link>
   <joint name="robot_footprint_joint" type="fixed">
@@ -268,5 +268,5 @@
     <visual name='hokuyo_visual'>
       <geometry>
-        <mesh filename="package://udacity_bot/meshes/hokuyo.dae" />
+        <mesh filename="package://slam_project/meshes/hokuyo.dae" />
       </geometry>
     </visual>
